File: JRT_relayBoard_Circuit/JRT_relayBoard_Circuit.kicad_pcb (KiCad board)
At the start: 2 copper layers, 100.2 x 63.6 mm, 8 parts, among them J1 Conn_ESP32_Left, J2 Conn_ESP32_Right, J3 eCON_D1-4, J4 eCON_D5-8, J5 eCON_D9-12, J6 eCON_D13-15, J7 eCON_A1-4, J8 eCON_A5_UART_Vin_Vout

Commit message: 電源スイッチ取付用穴を追加
Parts:
- added J9: PowerSwitch, Connector_PinSocket_2.54mm:PinSocket_1x03_P2.54mm_Vertical, F.Cu at (155.5, 143.5)
Connections:
- J2 pad 1: +9V -> +9VA
Routing:
- net +9VA: track 0.00 -> 60.3 mm
- net +9V: track 87.9 -> 28.8 mm
Other:
- board text added: "OFF"
- board text added: "ON"
